File: fch7.kicad_sch (KiCad schematic)
At the start: 0 parts

Commit message: update : pin stm32 connections
Parts:
- added C1: 2.2u, symbol Device:C
- added R1: 10k, symbol Device:R
- added R2, R3: 2.2k, symbol Device:R
- added SW1: SW_Push_Open, symbol Switch:SW_Push_Open
- added U1: STM32H743VITx, Package_QFP:LQFP-100_14x14mm_P0.5mm, symbol MCU_ST_STM32H7:STM32H743VITx
Connections:
- new net: C1.1, U1.48 (VCAP), U1.73 (VCAP)
- new net: R1.2, SW1.2 (B), U1.94 (BOOT0)
- new net AIRS: U1.32 (PC4)
- new net BEEPER: U1.77 (PA15)
- new net CAN RX: U1.82 (PD1)
- new net CAN TX: U1.81 (PD0)
- new net EXTI CS1: U1.85 (PD4)
- new net GND: C1.2, R1.1, U1.10 (VSS), U1.26 (VSS), U1.49 (VSS), U1.74 (VSS), U1.99 (VSS)
- new net I2C1 CLK: R2.1, U1.92 (PB6)
- new net I2C1 SDA: R3.1, U1.93 (PB7)
- new net OTG FS_DM: U1.70 (PA11)
- new net OTG FS_DP: U1.71 (PA12)
- new net PWM SW_2812: U1.67 (PA8)
- new net PWM_10: U1.62 (PD15)
- new net PWM_7: U1.59 (PD12)
- new net PWM_8: U1.60 (PD13)
- new net PWM_9: U1.61 (PD14)
- new net RSSI: U1.33 (PC5)
- new net RX: U1.95 (PB8), U1.96 (PB9), U1.97 (PE0), U1.98 (PE1)
- new net SDIO CMD: U1.83 (PD2)
- new net SDIO_CLK: U1.80 (PC12)
- new net SDIO_D1: U1.65 (PC8), U1.66 (PC9)
- new net SDIO_D2: U1.78 (PC10)
- new net SDIO_D3: U1.79 (PC11)
- new net SPI1 MOSI: U1.88 (PD7)
- new net SPI2_MISO: U1.53 (PB14)
- new net SPI2_MOSI: U1.54 (PB15)
- new net SPI2_OSD_CS: U1.51 (PB12)
- new net SPI2_SCLK: U1.52 (PB13)
- new net SPI3 MISO: U1.90 (PB4)
- new net SPI3 MOSI: U1.91 (PB5)
- new net SPI3 SCLK: U1.89 (PB3)
- new net SWD SWCLK: U1.76 (PA14)
- new net SWD SWDIO: U1.72 (PA13)
- new net SW_CAMERA: U1.58 (PD11)
- new net SW_POWER: U1.57 (PD10)
- new net UART1_RX: U1.69 (PA10)
- new net UART1_TX: U1.68 (PA9)
- new net UART2 RX: U1.87 (PD6)
- new net UART2 TX: U1.86 (PD5)
- new net UART3_RX: U1.56 (PD9)
- new net UART3_TX: U1.55 (PD8)
- new net UART6_RX: U1.64 (PC7)
- new net UART6_TX: U1.63 (PC6)
- new net VDD_MCU: R2.2, R3.2, SW1.1 (A), U1.100 (VDD), U1.11 (VDD), U1.20 (VREF+), U1.21 (VDDA), U1.27 (VDD), U1.50 (VDD), U1.75 (VDD)
- no-connect marks 0 -> 2

Commit message: finished MCU sheet and start hierarchy sheets for other components
Parts:
- removed C1: 2.2u, symbol Device:C
- removed R1: 10k, symbol Device:R
- removed R2, R3: 2.2k, symbol Device:R
- removed SW1: SW_Push_Open, symbol Switch:SW_Push_Open
- removed U1: STM32H743VITx, Package_QFP:LQFP-100_14x14mm_P0.5mm, symbol MCU_ST_STM32H7:STM32H743VITx
Connections:
- no-connect marks 2 -> 0
Other:
- added sheet MCU (MCU.kicad_sch)
- added sheet Power (untitled.kicad_sch)
