File: fch7.kicad_sch (KiCad schematic)
At the start: 0 parts

Commit message: finished -power and sensors page, started OSD
Other:
- added sheet OSD (osd.kicad_sch)
- added sheet Sensors (sensors.kicad_sch)
Changed lines of the file:
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@@
+		)
+	)
+	(sheet
+		(at -179.07 64.77)
+		(size 99.06 151.13)
+		(exclude_from_sim no)
+		(in_bom yes)
+		(on_board yes)
+		(dnp no)
+		(fields_autoplaced yes)
+		(stroke
+			(width 0.1524)
+			(type solid)
+		)
+		(fill
+			(color 0 0 0 0.0000)
+		)
+		(property "Sheetname" "OSD"
+			(at -179.07 64.0584 0)
+			(effects
+				(font
+					(size 1.27 1.27)
+				)
+				(justify left bottom)
+			)
+		)
+		(property "Sheetfile" "osd.kicad_sch"
+			(at -179.07 216.4846 0)
+			(effects
+				(font
+					(size 1.27 1.27)
+				)
+				(justify left top)
+			)
+		)
+		(instances
+			(project "fch7"
+				(path "/11716af6-0e6e-444b-b738-3f12da23c1a2"
+					(page "5")
+				)
+			)
+		)
+	)
+	(sheet
+		(at 444.5 247.65)
+		(size 318.77 231.14)
+		(exclude_from_sim no)
+		(in_bom yes)
+		(on_board yes)
+		(dnp no)
+		(fields_autoplaced yes)
+		(stroke
+			(width 0.1524)
+			(type solid)
+		)
+		(fill
+			(color 0 0 0 0.0000)
+		)
+		(property "Sheetname" "Sensors"
+			(at 444.5 246.9384 0)
+			(effects
+				(font
+					(size 1.27 1.27)
+				)
+				(justify left bottom)
+			)
+		)
+		(property "Sheetfile" "sensors.kicad_sch"
+			(at 444.5 479.3746 0)
+			(effects
+				(font
+					(size 1.27 1.27)
+				)
+				(justify left top)
+			)
+		)
+		(instances
+			(project "fch7"
+				(path "/11716af6-0e6e-444b-b738-3f12da23c1a2"
+					(page "4")
+				)
+			)
 		)
 	)

Commit message: finished blackbox led and osd, then started rx
Other:
- added sheet Blackbox_led (blackbox_led.kicad_sch)
- added sheet wifi (wifi.kicad_sch)
Changed lines of the file:
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@@
+		)
+	)
+	(sheet
+		(at -242.57 -157.48)
+		(size 242.57 124.46)
+		(exclude_from_sim no)
+		(in_bom yes)
+		(on_board yes)
+		(dnp no)
+		(fields_autoplaced yes)
+		(stroke
+			(width 0.1524)
+			(type solid)
+		)
+		(fill
+			(color 0 0 0 0.0000)
+		)
+		(property "Sheetname" "wifi"
+			(at -242.57 -158.1916 0)
+			(effects
+				(font
+					(size 1.27 1.27)
+				)
+				(justify left bottom)
+			)
+		)
+		(property "Sheetfile" "wifi.kicad_sch"
+			(at -242.57 -32.4354 0)
+			(effects
+				(font
+					(size 1.27 1.27)
+				)
+				(justify left top)
+			)
+		)
+		(instances
+			(project "fch7"
+				(path "/11716af6-0e6e-444b-b738-3f12da23c1a2"
+					(page "7")
+				)
+			)
+		)
+	)
+	(sheet
+		(at 76.2 -177.8)
+		(size 508 140.97)
+		(exclude_from_sim no)
+		(in_bom yes)
+		(on_board yes)
+		(dnp no)
+		(fields_autoplaced yes)
+		(stroke
+			(width 0.1524)
+			(type solid)
+		)
+		(fill
+			(color 0 0 0 0.0000)
+		)
+		(property "Sheetname" "Blackbox_led"
+			(at 76.2 -178.5116 0)
+			(effects
+				(font
+					(size 1.27 1.27)
+				)
+				(justify left bottom)
+			)
+		)
+		(property "Sheetfile" "blackbox_led.kicad_sch"
+			(at 76.2 -36.2454 0)
+			(effects
+				(font
+					(size 1.27 1.27)
+				)
+				(justify left top)
+			)
+		)
+		(instances
+			(project "fch7"
+				(path "/11716af6-0e6e-444b-b738-3f12da23c1a2"
+					(page "6")
+				)
+			)
 		)
 	)

Commit message: finshed every schematic pages, remains footprints assignments
Other:
- sheet wifi renamed rf_rx
- added sheet connectors (connectors.kicad_sch)
- sheet rf_rx: file wifi.kicad_sch -> rf_rx.kicad_sch
Changed lines of the file:
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@@
+	)
+	(sheet
+		(at 650.24 -109.22)
+		(size 248.92 86.36)
+		(exclude_from_sim no)
+		(in_bom yes)
+		(on_board yes)
+		(dnp no)
+		(fields_autoplaced yes)
+		(stroke
+			(width 0.1524)
+			(type solid)
+		)
+		(fill
+			(color 0 0 0 0.0000)
+		)
+		(property "Sheetname" "connectors"
+			(at 650.24 -109.9316 0)
+			(effects
+				(font
+					(size 1.27 1.27)
+				)
+				(justify left bottom)
+			)
+		)
+		(property "Sheetfile" "connectors.kicad_sch"
+			(at 650.24 -22.2754 0)
+			(effects
+				(font
+					(size 1.27 1.27)
+				)
+				(justify left top)
+			)
+		)
+		(instances
+			(project "fch7"
+				(path "/11716af6-0e6e-444b-b738-3f12da23c1a2"
+					(page "8")
+				)
+			)
+		)
 	)
 	(sheet
@@
 			(color 0 0 0 0.0000)
 		)
-		(property "Sheetname" "wifi"
+		(property "Sheetname" "rf_rx"
 			(at -242.57 -158.1916 0)
 			(effects
@@
 			)
 		)
-		(property "Sheetfile" "wifi.kicad_sch"
+		(property "Sheetfile" "rf_rx.kicad_sch"
 			(at -242.57 -32.4354 0)
 			(effects
